File: hw/boards/tk1/tk1.kicad_pcb (KiCad board)
At the start: 4 copper layers, 27.5 x 13.5 mm, 68 parts, among them P1 USB_C_Plug, U1 MCP1824T-2502EOT, U10 PT2043AT6, U2 MIC5258-1.2YM5, U3 CH552E, U5 USBLC6-2SC6, U6 ICE40UP5K-SG48ITR, U8 XT25F08BDFIGT-S, U9 NCP752BSN33T1G

Commit message: TK-1 and TP-1 PCBs (#52)
* Add kicad library for flat programming clip

* Add descriptions to part symbols

* Add extended values, manufacturer/distributor info to components in mta1

* Add new board entry for TK1

* Add TP1 programmer design

* Update MTA1-USB-V1 release files to match production

* Change SPI flash memory type to XT25F08BDFIGT-S
* Change touch sensor feedback cap to 1uF
* Add manufacturer, manufacturer part number, distributor, distributor part number

* Update component values for TK1 PCB

* Use specific part # for C8
* Change flash back to Winbond part, for easier sourcing
* Change C1 to 1pF

* Fixes for production programmer PCB

* Swap GND and 5V on J3
* Replace graphic logo with text
* Rename part to 'TP-1'

* TK-1 release

* Add dimensions for PCB
* Add layer stackup for PCB
* Change PCB component origin to match expanded board
* Change schematic title to 'TK-1', update release date

* mta1-usb-v1-programmer: Add corrected part numbers for OSFC production

* Q1, Q2, F1 part subsititutions
* add mfr/supplier info for all parts

* PCB library: add parts

* Rectangular footprint for TK-1 test pads
* BOM generation script used for TK-1 and TP-1 releases

* TP-1 release

* Schematic: Add manufacturer, supplier information for all parts
* Schematic: Update name and release date
* PCB: Add PCB fabrication information
* PCB: Correct pinouts on silkscreen

* PCB library: add 'screw' and 'foot' symbols

* Screw is a schematic-only part, for including mechanical screws in the
  BOM
* Foot is for self-adhesive rubber mounting feet that can be stuck to
  the bottom of a PCB

* TP-1 release: Add screws, feet to the BOM

* Pico library: Add footprint for RPi Pico w/solder paste

* TP-1 RevA release updates:

* Add fiducials in 3 corners (1mm exposed copper ring w/2mm soldermask opening)
* Add solder paste openings to Raspberry Pi Pico pads

* TK-1: RevA.1 release

* Add two fiducials to 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
Parts:
- added FID1: Fiducial, Fiducial:Fiducial_0.75mm_Mask1.5mm, F.Cu at (101.5, 88.5)
- added FID2: Fiducial, Fiducial:Fiducial_0.75mm_Mask1.5mm, F.Cu at (124.2, 96.8)
- C27: value 2.7pF -> 1pF
- C8: value 10uF -> 1uF
- TP1, TP12, TP13, TP14, TP15, TP16, TP17, TP18, TP19, TP2, TP20, TP21, TP28, TP3, TP4, TP5, TP6, TP7, TP8, TP9: footprint TestPoint:TestPoint_Pad_D1.0mm -> mta1:TestPoint_Pad_D1.0mm
- U8: value XT25F08BDFIGT-S -> W25Q80DVUXIE
- turned TP1 to 0 degrees
- turned TP2 to 180 degrees
- turned TP3 to 0 degrees
- turned TP4 to 0 degrees
Routing:
- net GND: track 38.0 -> 39.6 mm, vias 38 -> 37
- net APP_ICE_MISO: track 9.88 -> 8.46 mm
- net +3V3: track 36.7 -> 37.8 mm
- net INTERFACE_RX: track 10.1 -> 11.0 mm
- net INTERFACE_CTS: track 8.98 -> 8.38 mm
- net +2V5: track 17.3 -> 17.8 mm
Other:
- board size 27.5 x 13.5 mm -> 27.7 x 13.9 mm
- board text added: "0"
- board text added: "0 mm"
- board text added: "0.01 mm"
- board text added: "0.0175 mm"
- board text added: "0.02"
- board text added: "0.035 mm"
- board text added: "0.121 mm"
- board text added: "0.433 mm"
- board text added: "1"
- board text added: "2022-11 RevA"
- board text added: "3.3"
- board text added: "4.5"
- board text added: "B.Cu"
- board text added: "B.Mask"
- board text added: "B.Paste"
- board text added: "B.Silkscreen"
- board text added: "Black"
- board text added: "Bottom Silk Screen"
- board text added: "Bottom Solder Mask"
- board text added: "Bottom Solder Paste"
- board text added: "Color"
- board text added: "Dielectric 1"
- board text added: "Dielectric 2"
- board text added: "Dielectric 3"
- board text added: "Epsilon R"
- board text added: "F.Cu"
- board text added: "F.Mask"
- board text added: "F.Paste"
- board text added: "F.Silkscreen"
- board text added: "FR4"
- board text added: "In1.Cu"
- board text added: "In2.Cu"
- board text added: "Layer Name"
- board text added: "Loss Tangent"
- board text added: "Material"
- board text added: "Not specified"
- board text added: "Thickness (mm)"
- board text added: "Tillitis TK-1"
- board text added: "Top Silk Screen"
- board text added: "Top Solder Mask"
- board text added: "Top Solder Paste"
- board text added: "Type"
- board text added: "White"
- board text added: "copper"
- board text added: "core"
- board text added: "prepreg"
- board text removed: "+1.2V"
- board text removed: "+2.5V"
- board text removed: "+3.3V"
- board text removed: "+5V"
- board text removed: "MTA1-USB V1"
- board text removed: "Test pads on bottom:"
