File: hw/application_fpga.kicad_sch (KiCad schematic)
At the start: 39 parts, among them U10 PT2043AT6, U6 ICE40UP5K-SG48ITR, U8 W25Q80DVUXIE

Commit message: Update project links to library
- Symbols
- Footprints
- Draw sheet
Parts:
- C8: value (none) -> 1uF; footprint (none) -> Capacitor_SMD:C_1206_3216Metric
- U11: value (none) -> ~
Other:
- title: Application FPGA -> TK-1

Commit message: Fix all ERC errors
- Update symbols
- Add PWR_FLAG
- Disable error on SPICE models
Parts:
- U11: footprint (none) -> 1674954-1
Connections:
- net +3V3 renamed +3.3V
Changed lines of the file:
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@@
   (junction (at 203.2 101.6) (diameter 0) (color 0 0 0 0)
+  )
+  (junction (at 35.56 45.72) (diameter 0) (color 0 0 0 0)
   )
   (junction (at 41.91 35.56) (diameter 0) (color 0 0 0 0)
@@
     (stroke (width 0) (type default))
   )
+  (wire (pts (xy 35.56 45.72) (xy 41.91 45.72))
+    (stroke (width 0) (type default))
+  )
   (polyline (pts (xy 238.76 113.03) (xy 278.13 113.03))
     (stroke (width 0) (type solid))
@@
     (stroke (width 0) (type default))
   )
-  (wire (pts (xy 33.02 45.72) (xy 41.91 45.72))
+  (wire (pts (xy 33.02 45.72) (xy 35.56 45.72))
     (stroke (width 0) (type default))
   )
@@
     )
     (property "Supplier Part Number" "220-2145-2-ND" (at 104.14 91.44 0)
+      (effects (font (size 1.27 1.27)) hide)
+    )
+    (property "Component" "" (at 104.14 91.44 0)
+      (effects (font (size 1.27 1.27)) hide)
+    )
+    (property "Rating" "" (at 104.14 91.44 0)
+      (effects (font (size 1.27 1.27)) hide)
+    )
+    (property "Package" "" (at 104.14 91.44 0)
+      (effects (font (size 1.27 1.27)) hide)
+    )
+    (property "Or equivalent" "" (at 104.14 91.44 0)
       (effects (font (size 1.27 1.27)) hide)
     )
@@
       (effects (font (size 1.27 1.27)) hide)
     )
+    (property "Component" "" (at 29.21 45.72 0)
+      (effects (font (size 1.27 1.27)) hide)
+    )
+    (property "Rating" "" (at 29.21 45.72 0)
+      (effects (font (size 1.27 1.27)) hide)
+    )
+    (property "Package" "" (at 29.21 45.72 0)
+      (effects (font (size 1.27 1.27)) hide)
+    )
+    (property "Or equivalent" "" (at 29.21 45.72 0)
+      (effects (font (size 1.27 1.27)) hide)
+    )
     (pin "1")
     (pin "2")
@@
     )
   )
+  (symbol (lib_id "power:PWR_FLAG") (at 35.56 45.72 0) (unit 1)
+    (in_bom yes) (on_board yes) (dnp no) (fields_autoplaced)
+    (property "Reference" "#FLG01" (at 35.56 43.815 0)
+      (effects (font (size 1.27 1.27)) hide)
+    )
+    (property "Value" "PWR_FLAG" (at 35.56 40.64 0)
+      (effects (font (size 1.27 1.27)) hide)
+    )
+    (property "Footprint" "" (at 35.56 45.72 0)
+      (effects (font (size 1.27 1.27)) hide)
+    )
+    (property "Datasheet" "~" (at 35.56 45.72 0)
+      (effects (font (size 1.27 1.27)) hide)
+    )
+    (pin "1")
+    (instances
+      (project "tk1"
+        (path "/8fc062a7-114d-48eb-a8f8-71128838f380/00000000-0000-0000-0000-00006161400b"
+          (reference "#FLG01") (unit 1)
+        )
+        (path "/8fc062a7-114d-48eb-a8f8-71128838f380/00000000-0000-0000-0000-0000611cc101"
+          (reference "#FLG03") (unit 1)
+        )
+      )
+    )
+  )
   (symbol (lib_id "Connector:TestPoint") (at 36.83 139.7 0) (unit 1)
     (in_bom no) (on_board yes) (dnp no)
@@
       (effects (font (size 1.27 1.27)) (justify right))
     )
-    (property "Footprint" "" (at 185.42 71.12 0)
+    (property "Footprint" "1674954-1" (at 185.42 71.12 0)
       (effects (font (size 1.27 1.27)) (justify left) hide)
     )
