File: hw/powersupply.kicad_sch (KiCad schematic)
At the start: 19 parts, among them U1 MCP1824T-2502EOT, U2 MIC5258-1.2YM5, U9 NCP752BSN33T1G

Commit message: Update project links to library
- Symbols
- Footprints
- Draw sheet
Other:
- title: Power Supply -> TK-1

Commit message: Fix all ERC errors
- Update symbols
- Add PWR_FLAG
- Disable error on SPICE models
Connections:
- net +3V3 renamed +3.3V
Changed lines of the file:
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@@
+      (effects (font (size 1.27 1.27)) hide)
+    )
+    (property "Component" "" (at 64.77 45.72 0)
+      (effects (font (size 1.27 1.27)) hide)
+    )
+    (property "Rating" "" (at 64.77 45.72 0)
+      (effects (font (size 1.27 1.27)) hide)
+    )
+    (property "Package" "" (at 64.77 45.72 0)
+      (effects (font (size 1.27 1.27)) hide)
+    )
+    (property "Or equivalent" "" (at 64.77 45.72 0)
       (effects (font (size 1.27 1.27)) hide)
     )
@@
       (effects (font (size 1.27 1.27)) hide)
     )
+    (property "Component" "" (at 63.5 92.71 0)
+      (effects (font (size 1.27 1.27)) hide)
+    )
+    (property "Rating" "" (at 63.5 92.71 0)
+      (effects (font (size 1.27 1.27)) hide)
+    )
+    (property "Package" "" (at 63.5 92.71 0)
+      (effects (font (size 1.27 1.27)) hide)
+    )
+    (property "Or equivalent" "" (at 63.5 92.71 0)
+      (effects (font (size 1.27 1.27)) hide)
+    )
